File: kicad/sirius.kicad_sch (KiCad schematic)
At the start: 5 parts

Commit message: Work on schematic some more
Parts:
- added C1, C2: 100n, Capacitor_SMD:C_0603_1608Metric, symbol Device:C_Small
- added C3: 100n, symbol Device:C_Small
- added D1, D2, D3: Green LED, symbol Device:LED
- added R1: 10k, symbol Device:R
- added R2, R3, R4: 1k, symbol Device:R_Small
- added SW1: SW_Push, symbol Switch:SW_Push
- GPS-RTK-Rover1: value LC29H -> LC29H (DA); footprint sirius:LC29H -> LC29H:XCVR_LC29H; symbol sirius:LC29H -> sirius:LC29H (DA); SNAPEDA_PN LC29H -> LC29H (DA)
Connections:
- net +3V3: now reaches LoRa_Radio_Module1.13 (3.3V)
- net +3V3: now also Flight_Computer1.1 (3V3_1), GPS-RTK-Rover1.22 (V_BCKP), GPS-RTK-Rover1.23 (VCC), IMU1.5 (VDDIO), IMU1.8 (VDD), C1.1, C2.1, R1.1, R3.2, R4.2
- net MISO: now reaches LoRa_Radio_Module1.2 (MISO)
- net MISO: now also Flight_Computer1.21 (GPIO9/SPI_MISO)
- net MOSI: now reaches LoRa_Radio_Module1.3 (MOSI)
- net MOSI: now also Flight_Computer1.19 (GPIO10/SPI_MOSI)
- net SCK: now reaches LoRa_Radio_Module1.4 (SCK)
- net SCK: now also Flight_Computer1.23 (GPIO11/SPI_SCLK)
- net CS0: now reaches LoRa_Radio_Module1.5 (NSS)
- net CS0: now also Flight_Computer1.24 (GPIO8/SPI_~{CE0})
- net RESET: now reaches LoRa_Radio_Module1.6 (RESET)
- net RESET: now also Flight_Computer1.11 (GPIO17/GPIO_GEN0)
- net GND: now reaches IMU1.6 (GND)
- net GND: now also Flight_Computer1.39 (GND_39), GPS-RTK-Rover1.10 (GND), GPS-RTK-Rover1.12 (GND__1), GPS-RTK-Rover1.13 (GND__2), GPS-RTK-Rover1.24 (GND__3), LoRa_Radio_Module1.8 (GND), Pressure_Sensor1.3 (VSS), C1.2, C2.2, C3.2, D1.1 (K), SW1.2
- net GPS_TX: now reaches GPS-RTK-Rover1.20 (TXD1)
- net GPS_TX: now also Flight_Computer1.10 (GPIO15/RXD0), D2.1 (K)
- net GPS_RX: now reaches GPS-RTK-Rover1.21 (RXD1)
- net GPS_RX: now also Flight_Computer1.8 (GPIO14/TXD0), D3.1 (K)
- net PPS: now reaches GPS-RTK-Rover1.3 (1PPS)
- net PPS: now also R2.1
- net at GPS-RTK-Rover1.8 (~{RESET}): now also C3.1, R1.2, SW1.1
- new net: D1.2 (A), R2.2
- new net: D2.2 (A), R3.1
- new net: D3.2 (A), R4.1
- now unconnected: LoRa_Radio_Module1.1 (GND), LoRa_Radio_Module1.10 (GND)
- no-connect marks 0 -> 16
Other:
- note added: "BMP581"
- note added: "ICM-45686"
- note added: "LC29H(DA)"
- note added: "LED's"
- note added: "Pi Zero 2W"
- note added: "RFM95-915S2"
- moved on the sheet: Flight_Computer1, IMU1, Pressure_Sensor1

Commit message: Work on schematic some more, only thing left is screw switch
Parts:
- added C1, C2: 100n, Capacitor_SMD:C_0603_1608Metric, symbol Device:C_Small
- added C12: 10u, symbol Device:C_Small
- added C13, C8: 100n, symbol Device:C_Small
- added C14: 33p, symbol Device:C_Small
- added C3, C4: 0, symbol Device:C_Small
- added C6, C7: 100p, symbol Device:C_Small
- added C9: 1n, symbol Device:C_Small
- added D4, D5: SP3205-01ETG, Diode_SMD:D_SOD-882, symbol Diode:PTVS5V0Z1USK
- added J1: IPEX_MHF1, sirius:ipex_mhf1, symbol sirius:IPEX_MHF1
- added L1: 68u, symbol Device:L_Small
- added R5: 0, symbol Device:R_Small
- added R6: 10r, symbol Device:R_Small
- renumbered C1 to C10, C2 to C11, C3 to C5, D2 to D1, D3 to D2, D1 to D3, R2 to R1, R3 to R2, R4 to R3, R1 to R4
Connections:
- net MISO is gone; now on net MISO_SPI0: Flight_Computer1.21 (GPIO9/SPI_MISO), LoRa_Radio_Module1.2 (MISO)
- net MOSI is gone; now on net MOSI_SPI0: Flight_Computer1.19 (GPIO10/SPI_MOSI), LoRa_Radio_Module1.3 (MOSI)
- net SCK is gone; now on net SCK_SPI0: Flight_Computer1.23 (GPIO11/SPI_SCLK), LoRa_Radio_Module1.4 (SCK)
- net +3V3: now also Flight_Computer1.17 (3V3_17), Pressure_Sensor1.1 (VDDIO), Pressure_Sensor1.10 (VDD), C1.1, C12.2, C13.2, C14.2, C2.2, D5.1 (K)
- net GND: now also Flight_Computer1.14 (GND_14), Flight_Computer1.20 (GND_20), Flight_Computer1.25 (GND_25), Flight_Computer1.30 (GND_30), Flight_Computer1.34 (GND_34), Flight_Computer1.6 (GND_6), Flight_Computer1.9 (GND_9), LoRa_Radio_Module1.1 (GND), LoRa_Radio_Module1.10 (GND), Pressure_Sensor1.8 (VSS), Pressure_Sensor1.9 (VSS), C1.2, C12.1, C13.1, C14.1, C2.1, C3.1, C4.1, C7.2, C8.2, C9.2, D4.2 (A), D5.2 (A), J1.2, J1.3
- net MISO_SPI1: now reaches IMU1.1 (AP_SDO/AP_AD0)
- net MISO_SPI1: now also Flight_Computer1.35 (GPIO19)
- net CS0_SPI1: now reaches IMU1.12 (AP_CS)
- net CS0_SPI1: now also Flight_Computer1.12 (GPIO18/GPIO_GEN1)
- net SCK_SPI1: now reaches IMU1.13 (AP_SCL/AP_SCLK)
- net SCK_SPI1: now also Flight_Computer1.40 (GPIO21)
- net MOSI_SPI1: now reaches IMU1.14 (AP_SDA/APSDIO/APSDI)
- net MOSI_SPI1: now also Flight_Computer1.38 (GPIO20)
- net SCK_SPI0: now reaches Pressure_Sensor1.2 (SCK)
- net MOSI_SPI0: now reaches Pressure_Sensor1.4 (SDI)
- net MISO_SPI0: now reaches Pressure_Sensor1.5 (SDO)
- net CS1_SPI0: now reaches Pressure_Sensor1.6 (CSB)
- net CS1_SPI0: now also Flight_Computer1.26 (GPIO7/SPI_~{CE1})
- net at GPS-RTK-Rover1.11 (RF_IN): now also C3.2, R5.1
- net VDD_RF: now reaches GPS-RTK-Rover1.9 (VDD_RF)
- net VDD_RF: now also C9.1, R6.2
- net +5V: now reaches Flight_Computer1.2 (5V_2)
- net +5V: now also Flight_Computer1.4 (5V_4)
- net CS0 renamed CS0_SPI0
- new net: C7.1, C8.1, L1.2, R6.1
- new net: C6.2, D4.1 (K), J1.1, L1.1
- new net: C4.2, C6.1, R5.2
- no-connect marks 16 -> 42
Other:
- note added: "Antenna will be soldered directly to ANT and GND pin."

Commit message: In progress Sirius PCB design
Parts:
- removed C10, C11: 100n, Capacitor_SMD:C_0603_1608Metric, symbol Device:C_Small
- removed C9: 1n, symbol Device:C_Small
- removed D5: SP3205-01ETG, Diode_SMD:D_SOD-882, symbol Diode:PTVS5V0Z1USK
- removed IMU1: ICM-45686, sirius:IC_ICM-45686, symbol sirius:ICM-45686
- removed Pressure_Sensor1: BMP581, sirius:BMP581, symbol sirius:BMP581
- removed R4: 10k, symbol Device:R
- removed SW1: SW_Push, symbol Switch:SW_Push
- added BZ1: Buzzer, sirius:CSS0575ASMTTR, symbol Device:Buzzer
- added C3: 10u, Capacitor_SMD:C_0603_1608Metric_Pad1.08x0.95mm_HandSolder, symbol Device:C_Small
- added C4: 100n, Capacitor_SMD:C_0603_1608Metric_Pad1.08x0.95mm_HandSolder, symbol Device:C_Small
- added C6: 44u, Capacitor_SMD:C_0603_1608Metric_Pad1.08x0.95mm_HandSolder, symbol Device:C_Small
- added C7: 1000u, Capacitor_SMD:CP_Elec_10x10.5, symbol Device:C_Polarized_Small
- added D1, D2, D4: LED_Small, LED_SMD:LED_0603_1608Metric_Pad1.05x0.95mm_HandSolder, symbol Device:LED_Small
- added D10: 1N4148W, Diode_SMD:D_SOD-123, symbol Diode:1N4148W
- added D5: Schottky, sirius:SOD-323HEUS2H_TOS, symbol Device:D_Schottky_Small
- added D6: 3.3V Zener, Package_TO_SOT_SMD:SOT-23-3, symbol Device:D_Zener_Small_Filled
- added J2: Power In, Connector_PinHeader_1.00mm:PinHeader_1x01_P1.00mm_Vertical, symbol Connector:Conn_01x01_Pin
- added J3: Screw_Terminal, TerminalBlock_Phoenix:TerminalBlock_Phoenix_MPT-0,5-2-2.54_1x02_P2.54mm_Horizontal, symbol Connector:Screw_Terminal_01x02
- added L1: 6.8u, sirius:1277AS-H-1R0M=P2, symbol Device:L_Small
- added Q1: Q_PMOS_GSD, sirius:SOT_7DS-T1-GE3_VIS, symbol Transistor_FET:Q_PMOS_GSD
- added Q2, Q3: Q_NMOS_GSD, Package_TO_SOT_SMD:TSOT-23, symbol Transistor_FET:Q_NMOS_GSD
- added R1: 2k, Resistor_SMD:R_0603_1608Metric_Pad0.98x0.95mm_HandSolder, symbol Device:R_Small
- added R10: 5.6k, Resistor_SMD:R_0603_1608Metric_Pad0.98x0.95mm_HandSolder, symbol Device:R_Small
- added R12: 10k, Resistor_SMD:R_0603_1608Metric_Pad0.98x0.95mm_HandSolder, symbol Device:R_Small
- added R13, R7: 1k, Resistor_SMD:R_0603_1608Metric_Pad0.98x0.95mm_HandSolder, symbol Device:R_Small
- added R16: 180R, Resistor_SMD:R_0603_1608Metric_Pad0.98x0.95mm_HandSolder, symbol Device:R_Small
- added R2: 158k, Resistor_SMD:R_0603_1608Metric_Pad0.98x0.95mm_HandSolder, symbol Device:R_Small
- added R3: 30.1k, Resistor_SMD:R_0603_1608Metric_Pad0.98x0.95mm_HandSolder, symbol Device:R_Small
- added R6: 1.2k, Resistor_SMD:R_0603_1608Metric_Pad0.98x0.95mm_HandSolder, symbol Device:R_Small
- added R8: 3.3k, Resistor_SMD:R_0603_1608Metric_Pad0.98x0.95mm_HandSolder, symbol Device:R_Small
- added R9: 100R, Resistor_SMD:R_0603_1608Metric_Pad0.98x0.95mm_HandSolder, symbol Device:R_Small
- added U1: Power_Connector, sirius:XT60, symbol sirius:XT60
- added U2: AP63301WU-7, sirius:SOT95P280X100-6N, symbol sirius:AP63300WU-7
- C1, C2: value 100n -> 10u; footprint Capacitor_SMD:C_0603_1608Metric -> Capacitor_SMD:C_0603_1608Metric_Pad1.08x0.95mm_HandSolder; Digikey PN 399-C0603C104K5RACTUCT-ND -> (none); MPN C1590 -> (none)
- C10: renamed from C6; footprint (none) -> Capacitor_SMD:C_0603_1608Metric
- C11: renamed from C7; footprint (none) -> Capacitor_SMD:C_0603_1608Metric
- C12: renamed from C8; footprint (none) -> Capacitor_SMD:C_0603_1608Metric
- C13: renamed from C12; footprint (none) -> Capacitor_SMD:C_0603_1608Metric
- C14: renamed from C13; footprint (none) -> Capacitor_SMD:C_0603_1608Metric
- C15: renamed from C14; footprint (none) -> Capacitor_SMD:C_0603_1608Metric
- C5: value 100n -> 47p; footprint (none) -> Capacitor_SMD:C_0603_1608Metric_Pad1.08x0.95mm_HandSolder
- C8: renamed from C3; footprint (none) -> Capacitor_SMD:C_0603_1608Metric; now not fitted
- C9: renamed from C4; footprint (none) -> Capacitor_SMD:C_0603_1608Metric; now not fitted
- D3: renamed from D4; value SP3205-01ETG -> TVS; Digikey PN (none) -> F9320CT-ND
- D7: renamed from D1; value Green LED -> Blue LED; footprint (none) -> LED_SMD:LED_0603_1608Metric_Pad1.05x0.95mm_HandSolder; Digikey PN (none) -> LTST-C194TBKT
- D8: renamed from D2; value Green LED -> Yellow LED; footprint (none) -> LED_SMD:LED_0603_1608Metric_Pad1.05x0.95mm_HandSolder; Digikey PN (none) -> 404-1273-1-ND
- D9: renamed from D3; value Green LED -> Orange LED; footprint (none) -> LED_SMD:LED_0603_1608Metric_Pad1.05x0.95mm_HandSolder; Digikey PN (none) -> 350-5990030137FCT-ND
- J1: MAXIMUM_PACKAGE_HEIGHT 1.25mm -> (none); MF I-PEX -> (none); MP 20279-001E-03 -> (none); PARTREV 32 -> (none)
- L2: renamed from L1; value 68u -> 68n; footprint (none) -> Inductor_SMD:L_0603_1608Metric
- R11: renamed from R1; footprint (none) -> Resistor_SMD:R_0603_1608Metric
- R14: renamed from R2; footprint (none) -> Resistor_SMD:R_0603_1608Metric
- R15: renamed from R3; footprint (none) -> Resistor_SMD:R_0603_1608Metric
- R4: renamed from R5; footprint (none) -> Resistor_SMD:R_0603_1608Metric
- R5: renamed from R6; footprint (none) -> Resistor_SMD:R_0603_1608Metric
- U4: renamed from GPS-RTK-Rover1; footprint LC29H:XCVR_LC29H -> sirius:LC29H; MANUFACTURER Quectel -> (none); MAXIMUM_PACKAGE_HEIGHT 2.70mm -> (none); PARTREV 1.1 -> (none); SNAPEDA_PN LC29H (DA) -> (none); STANDARD Manufacturer Recommendations -> (none)
- U5: renamed from Flight_Computer1; footprint sirius:pi_zero_2w -> sirius:Pi_hat_generic
- renumbered LoRa_Radio_Module1 to U3
Connections:
- net +3V3: now also BZ1.1 (+), D10.1 (K); no longer C1.1, C2.2
- net +5V: now also C5.1, C6.1, L1.2, R2.1
- net GND: now also C2.2, C3.2, C6.2, C7.2, D1.2 (A), D2.1 (K), D4.1 (K), D6.1 (A), Q1.1 (G), Q2.2 (S), Q3.2 (S), R10.2, R12.2, R3.2, U1.2 (Ground), U2.4 (GND); no longer C2.1, C5.2
- net GPIO25: now reaches U3.14 (DIO0)
- net GPIO25: now also U5.22 (GPIO25/GPIO_GEN6)
- net GPIO6: now reaches U3.15 (DIO1)
- net GPIO6: now also U5.31 (GPIO6)
- net GPIO26: now reaches U3.16 (DIO2)
- net GPIO26: now also U5.37 (GPIO26)
- net at U4.8 (~{RESET}): no longer C5.1
- net RF_IN: now reaches C8.2, R4.1, U4.11 (RF_IN)
- net CONTINUITY_SENSE: now reaches U5.13 (GPIO27/GPIO_GEN2)
- net CONTINUITY_SENSE: now also D6.3 (K), R8.1
- net PYRO_FIRE: now reaches U5.15 (GPIO22/GPIO_GEN3)
- net PYRO_FIRE: now also R12.1, R9.2
- net CS0_SPI1 renamed BUZZER_PIN
- net BUZZER_PIN: now also R16.1
- net CS1_SPI0: no longer names the net of U5.26 (GPIO7/SPI_~{CE1})
- net GPS_RX renamed Pi_TX
- net Pi_TX: now also R13.2; no longer U4.21 (RXD1)
- net GPS_TX renamed Pi_RX
- net Pi_RX: now also R7.1; no longer U4.20 (TXD1)
- net MISO_SPI1: no longer names the net of U5.35 (GPIO19)
- net MOSI_SPI1: no longer names the net of U5.38 (GPIO20)
- net SCK_SPI1: no longer names the net of U5.40 (GPIO21)
- new net: Q2.1 (G), R9.1
- new net: BZ1.2 (-), D10.2 (A), Q3.3 (D)
- new net: Q3.1 (G), R16.2
- new net: C5.2, R2.2, R3.1, U2.1 (FB)
- new net: D1.1 (K), D2.2 (A), R1.2
- new net: C4.2, L1.1, U2.5 (SW)
- new net: C4.1, U2.6 (BST)
- new net: D5.2 (A), J2.1 (Pin_1)
- new net: D4.2 (A), R6.2
- new net: R7.2, U4.20 (TXD1)
- new net +BATT: Q1.3 (D), R1.1, U1.1 (Vin)
- new net PYRO_NEGATIVE: J3.1 (Pin_1), Q2.3 (D), R6.1, R8.2
- new net PYRO_POSITIVE: D5.1 (K), J3.2 (Pin_2)
- new net Pi_TX_2_8: R10.1, R13.1, U4.21 (RXD1)
- new net VCC: C1.1, C2.1, C3.1, C7.1, Q1.2 (S), U2.2 (EN), U2.3 (VIN)
- no-connect marks 42 -> 30
Other:
- note added: "(from screw switch)"
- note added: "Activity Indicators"
- note added: "Bulk Capacitor"
- note added: "Buzzer"
- note added: "Continuity LED"
- note added: "Firing Circuit"
- note added: "IFA Antenna"
- note added: "Level Shifting"
- note added: "POWER"
- note added: "PYROTECHNICS"
- note added: "Pi Continuity Sensing"
- note added: "Power LED"
- note added: "Pyro Channel"
- note added: "RASPBERRY PI"
- note added: "RF"
- note added: "RP Protection"
- note added: "Terminals"
- note added: "Voltage Regulator"
- note added: "XT60 Power Connector"
- note removed: "Antenna will be soldered directly to ANT and GND pin."
- note removed: "BMP581"
- note removed: "ICM-45686"
- note removed: "LED's"
- moved on the sheet: C10, C11, C12, C13, C14, C15, D3, D7, D8, D9, J1, L2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

Commit message: Refactor to use classes properly
Recompile openEMS with boost 1.90 and link wheels. Also update the PCB with the antenna. Still unrouted
Parts:
- added C2, C5: 0, Capacitor_SMD:C_0603_1608Metric, symbol Device:C_Small
- added NT1: NetTie_2, sirius:IFA_915, symbol Device:NetTie_2
- added R1: 0, Resistor_SMD:R_0603_1608Metric, symbol Device:R_Small
- U3: DESCRIPTION RFM95W LoRA Transceiver Module 915MHz -> (none)
- renumbered C8 to C10, C9 to C11, C10 to C12, C11 to C13, C12 to C14, C13 to C15, C14 to C16, C15 to C17, C2 to C3, C3 to C4, C4 to C6, C5 to C7, C6 to C8, C7 to C9, R9 to R10, R10 to R11, R11 to R12, R12 to R13, R13 to R14, R14 to R15, R15 to R16, R16 to R17, R1 to R2, R2 to R3, R3 to R4, R4 to R5, R5 to R6, R6 to R7, R7 to R8, R8 to R9
Connections:
- net GND: now also C2.2, C5.2, NT1.1
- net at U3.9 (ANT): now also C5.1, R1.2
- new net: C2.1, NT1.2, R1.1
Other:
- note removed: "IFA Antenna"
- moved on the sheet: U3

Commit message: Finish Sirius PCB design
Logo pending
Changed lines of the file:
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@@
 		)
 	)
-	(label "VCC"
-		(at 109.22 34.29 0)
-		(effects
-			(font
-				(size 1.27 1.27)
-			)
-			(justify left bottom)
-		)
-	)
 	(label "RF_IN"
 		(at 133.35 175.26 0)
@@
 					(unit 1)
 				)
+			)
+		)
+	)
+	(symbol
+		(lib_id "power:VCC")
+		(at 109.22 34.29 0)
+		(unit 1)
+		(body_style 1)
+		(exclude_from_sim no)
+		(in_bom yes)
+		(on_board yes)
+		(in_pos_files yes)
+		(dnp no)
+		(property "Reference" "#PWR041"
+			(at 109.22 38.1 0)
+			(hide yes)
+			(show_name no)
+			(do_not_autoplace no)
+			(effects
+				(font
+					(size 1.27 1.27)
+				)
+			)
+		)
+		(property "Value" "VCC"
+			(at 109.22 30.226 0)
+			(show_name no)
+			(do_not_autoplace no)
+			(effects
+				(font
+					(size 1.27 1.27)
+				)
+			)
+		)
+		(property "Footprint" ""
+			(at 109.22 34.29 0)
+			(hide yes)
+			(show_name no)
+			(do_not_autoplace no)
+			(effects
+				(font
+					(size 1.27 1.27)
+				)
+			)
+		)
+		(property "Datasheet" ""
+			(at 109.22 34.29 0)
+			(hide yes)
+			(show_name no)
+			(do_not_autoplace no)
+			(effects
+				(font
+					(size 1.27 1.27)
+				)
+			)
+		)
+		(property "Description" "Power symbol creates a global label with name \"VCC\""
+			(at 109.22 34.29 0)
+			(hide yes)
+			(show_name no)
+			(do_not_autoplace no)
+			(effects
+				(font
+					(size 1.27 1.27)
+				)
+			)
+		)
+		(pin "1"
+		)
+		(instances
+			(project "sirius"
+				(path "/abc76503-1c89-48c4-92f2-dcc55eacd272"
+					(reference "#PWR041")
+					(unit 1)
+				)
